Commit message: revised name from origin(xx1)

File: aip_axio_description/urdf/sensor_kit.xacro (robot description, xacro)
@@ -23,5 +23,5 @@
     <!-- lidar -->
     <VLP-16 parent="sensor_kit_base_link" name="velodyne_top" topic="/points_raw" hz="10" samples="220" gpu="$(arg gpu)">
-      <origin xyz="${calibration['sensor_kit_base_link2velodyne_left_top_link']['x']} ${calibration['sensor_kit_base_link2velodyne_top_base_link']['y']} ${calibration['sensor_kit_base_link2velodyne_top_base_link']['z']}" rpy="${calibration['sensor_kit_base_link2velodyne_top_base_link']['roll']} ${calibration['sensor_kit_base_link2velodyne_top_base_link']['pitch']} ${calibration['sensor_kit_base_link2velodyne_top_base_link']['yaw']}" />
+      <origin xyz="${calibration['sensor_kit_base_link2velodyne_top_base_link']['x']} ${calibration['sensor_kit_base_link2velodyne_top_base_link']['y']} ${calibration['sensor_kit_base_link2velodyne_top_base_link']['z']}" rpy="${calibration['sensor_kit_base_link2velodyne_top_base_link']['roll']} ${calibration['sensor_kit_base_link2velodyne_top_base_link']['pitch']} ${calibration['sensor_kit_base_link2velodyne_top_base_link']['yaw']}" />
     </VLP-16>
     <!-- camera -->
